Commit message: Fixed URDF, rviz

File: install/bot_description/share/bot_description/urdf/bot_urdf.urdf (robot description, URDF)
Before this commit: robot kartik_robot, 5 links, 4 joints
Links:
- removed link base_footprint
- removed link front_caster
- added link caster; collision sphere radius=0.03; visual sphere radius=0.03
- added link lwheel; visual cylinder length=0.008 radius=0.06
- added link rwheel; visual cylinder length=0.008 radius=0.06
- link base_link: geometry visual box size=0.2 0.2 0.1
- link camera_link: geometry visual box size=0.010 0 0.03
- link lidar_link: geometry collision cylinder length=0.1 radius=0.02; visual cylinder length=0.1 radius=0.02
Joints:
- removed joint base_joint
- added joint base_to_lwheel: type fixed, parent base_link, child lwheel, origin xyz=0 0.115 0.046 rpy=1.5708 0 0
- added joint base_to_rwheel: type fixed, parent base_link, child rwheel, origin xyz=0 -0.115 0.046 rpy=-1.5708 0 0
- joint camera_joint: origin xyz=0.305 0 0.08 rpy=0 0 0 -> xyz=0.06 0 0.2 rpy=0 0 0
- joint caster_joint: child front_caster -> caster; origin xyz=${caster_xoff} 0.0 ${-(base_height/2)} rpy=0 0 0 -> xyz=0.039 0.0 0.05 rpy=0 0 0
- joint lidar_joint: origin xyz=0.215 0 0.13 rpy=0 0 0 -> xyz=0.025 0 0.2 rpy=0 0 0

File: src/bot_description/urdf/bot_urdf.urdf (robot description, URDF)
Before this commit: robot kartik_robot, 5 links, 4 joints
Links:
- removed link base_footprint
- removed link front_caster
- added link caster; collision sphere radius=0.03; visual sphere radius=0.03
- added link lwheel; visual cylinder length=0.008 radius=0.06
- added link rwheel; visual cylinder length=0.008 radius=0.06
- link base_link: geometry visual box size=0.2 0.2 0.1
- link camera_link: geometry visual box size=0.010 0 0.03
- link lidar_link: geometry collision cylinder length=0.1 radius=0.02; visual cylinder length=0.1 radius=0.02
Joints:
- removed joint base_joint
- added joint base_to_lwheel: type fixed, parent base_link, child lwheel, origin xyz=0 0.115 0.046 rpy=1.5708 0 0
- added joint base_to_rwheel: type fixed, parent base_link, child rwheel, origin xyz=0 -0.115 0.046 rpy=-1.5708 0 0
- joint camera_joint: origin xyz=0.305 0 0.08 rpy=0 0 0 -> xyz=0.06 0 0.2 rpy=0 0 0
- joint caster_joint: child front_caster -> caster; origin xyz=${caster_xoff} 0.0 ${-(base_height/2)} rpy=0 0 0 -> xyz=0.039 0.0 0.05 rpy=0 0 0
- joint lidar_joint: origin xyz=0.215 0 0.13 rpy=0 0 0 -> xyz=0.025 0 0.2 rpy=0 0 0

Commit message: Added bot_world pkg

File: install/bot_description/share/bot_description/urdf/bot_urdf.urdf (robot description, URDF)
Before this commit: robot kartik_robot, 6 links, 5 joints
Joints:
- joint camera_joint: origin xyz=0.06 0 0.2 rpy=0 0 0 -> xyz=0.08 0 0.2 rpy=0 0 0
